Commit message: Vollständige Umgebung Kameras buggen 05.03 3:23

File: urdf/my_robot_description_V2.0.urdf (robot description, URDF)
Before this commit: robot my_robot, 14 links, 13 joints
Links:
- link base_link: geometry collision box size=3.5 2.0 0.5; visual mesh filename=package://my_robot_description/models/Oberteil.stl
- link base_wheel_left: geometry collision sphere radius=0.12; visual mesh filename=package://my_robot_description/models/Rad_links.stl
- link base_wheel_right: geometry collision sphere radius=0.12; visual mesh filename=package://my_robot_description/models/Rad_rechts.stl
- link camera_back: geometry visual mesh filename=package://my_robot_description/models/Kamera_hinten.stl
- link camera_back_floor: geometry visual mesh filename=package://my_robot_description/models/Kamera_hinten_unten.s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
- link camera_front: geometry visual mesh filename=package://my_robot_description/models/Kamera_vorne.stl
- link camera_front_floor: geometry visual mesh filename=package://my_robot_description/models/Kamera_vorne_unten.stl
- link camera_left: geometry visual mesh filename=package://my_robot_description/models/Kamera_links.stl
- link camera_right: geometry visual mesh filename=package://my_robot_description/models/Kamera_rechts.stl
- link lidar: geometry collision cylinder length=0.04 radius=0.05; visual mesh filename=package://my_robot_description/models/Lidar.stl
- link small_base: geometry collision box size=2.0 1.5 0.3; visual mesh filename=package://my_robot_description/models/Unterteil.stl
- link small_base_brush_left: geometry collision cylinder length=0.05 radius=0.15; visual mesh filename=package://my_robot_description/models/Buerste_links.stl
- link small_base_brush_right: geometry collision cylinder length=0.05 radius=0.15; visual mesh filename=package://my_robot_description/models/Buerste_rechts.stl
- link small_base_wheel_front: geometry collision sphere radius=0.12; visual mesh filename=package://my_robot_description/models/Rad_vorne.stl
Joints:
- joint brush_left_to_small_base: origin xyz=0.42 0.22 -0.37 rpy=0 0 0 -> xyz=1.05 0.55 -0.925 rpy=0 0 0
- joint brush_right_to_small_base: origin xyz=0.42 -0.22 -0.37 rpy=0 0 0 -> xyz=1.05 -0.55 -0.925 rpy=0 0 0
- joint lidar_to_base: origin xyz=-0.308 0 1.22 rpy=0 0 0 -> xyz=-0.77 0 3.05 rpy=0 0 0
- joint small_base_to_base: origin xyz=0.06 0.0 0.52 rpy=0 0 0 -> xyz=0.15 0 1.3 rpy=0 0 0
- joint wheel_front_to_small_base: origin xyz=-0.048 0.0 -0.416 rpy=0 0 0 -> xyz=-0.12 0 -1.04 rpy=0 0 0
- joint wheel_left_to_base: origin xyz=-0.636 0.26 0.104 rpy=0 0 0 -> xyz=-1.59 0.65 0.26 rpy=0 0 0
- joint wheel_right_to_base: origin xyz=-0.636 -0.26 0.104 rpy=0 0 0 -> xyz=-1.59 -0.65 0.26 rpy=0 0 0
