Commit message: Fahren gefixt, Kameras vorne bereit, autonomes fahren begonnen

File: urdf/my_robot_description.urdf (robot description, URDF)
Before this commit: robot my_robot, 14 links, 13 joints
Links:
- added link base_footprint
- link base_wheel_left: geometry collision cylinder length=0.05 radius=0.104; visual mesh filename=package://my_robot_description/models/Rad_links.stl scale=0.4 0.4 0.4
- link base_wheel_right: geometry collision cylinder length=0.05 radius=0.104; visual mesh filename=package://my_robot_description/models/Rad_rechts.stl scale=0.4 0.4 0.4
Joints:
- added joint base_footprint_to_base: type fixed, parent base_footprint, child base_link, origin xyz=0 0 0 rpy=0 0 0
- joint camera_back_floor_to_base: origin xyz=0 0 0 rpy=0 0 0 -> xyz=-0.77 0.01 0.4615 rpy=0 0.087 0
- joint camera_back_to_base: origin xyz=0 0 0 rpy=0 0 0 -> xyz=-0.765 0.01 0.56 rpy=0 0 0
- joint camera_front_floor_to_base: origin xyz=0 0 0 rpy=0 0 0 -> xyz=0.35 0.01 0.476 rpy=0 0 0
- joint camera_front_to_base: origin xyz=0 0 0 rpy=0 0 0 -> xyz=0.346 0.01 0.65 rpy=0 0 0
- joint camera_left_to_base: origin xyz=0 0 0 rpy=0 0 0 -> xyz=-0.33 0.318 0.56 rpy=0 0 -1.5708
- joint camera_right_to_base: origin xyz=0 0 0 rpy=0 0 0 -> xyz=-0.33 -0.293 0.56 rpy=0 0 0
- joint small_base_to_base: origin xyz=0.06 0.0 0.52 rpy=0 0 0 -> xyz=0.06 0 0.52 rpy=0 0 0
- joint wheel_front_to_small_base: origin xyz=-0.048 0.0 -0.416 rpy=0 0 0 -> xyz=-0.048 0 -0.416 rpy=0 0 0

Commit message: Kameras funktionieren alle

File: urdf/my_robot_description.urdf (robot description, URDF)
Before this commit: robot my_robot, 15 links, 14 joints
Joints:
- joint camera_back_floor_to_base: origin xyz=-0.77 0.01 0.4615 rpy=0 0.087 0 -> xyz=-0.77 -0.025 0.4615 rpy=0 0 3.1416
- joint camera_back_to_base: origin xyz=-0.765 0.01 0.56 rpy=0 0 0 -> xyz=-0.765 -0.025 0.56 rpy=0 0 3.1416
- joint camera_left_to_base: origin xyz=-0.33 0.318 0.56 rpy=0 0 -1.5708 -> xyz=-0.374 0.294 0.56 rpy=0 0 1.5708
- joint camera_right_to_base: origin xyz=-0.33 -0.293 0.56 rpy=0 0 0 -> xyz=-0.33 -0.32 0.56 rpy=0 0 -1.5708

Commit message: Alles Funktionen bereit

File: urdf/my_robot_description.urdf (robot description, URDF)
Before this commit: robot my_robot, 15 links, 14 joints
Links:
- link small_base: mass 3.0 -> 1.5
- link small_base_wheel_front: geometry collision cylinder length=0.05 radius=0.104; visual mesh filename=package://my_robot_description/models/Rad_vorne.stl scale=0.4 0.4 0.4
Joints:
- joint base_footprint_to_base: origin xyz=0 0 0 rpy=0 0 0 -> xyz=0 0 0.104 rpy=0 0 0
- joint wheel_left_to_base: origin xyz=-0.636 0.26 0.104 rpy=0 0 0 -> xyz=-0.636 0.241 0.104 rpy=0 0 0
- joint wheel_right_to_base: origin xyz=-0.636 -0.26 0.104 rpy=0 0 0 -> xyz=-0.636 -0.267 0.104 rpy=0 0 0

Commit message: Autonomes und manuelles fahren funktioniert

File: urdf/my_robot_description.urdf (robot description, URDF)
Before this commit: robot my_robot, 15 links, 14 joints
Links:
- link base_link: geometry collision box size=1.4 0.8 0.2; visual mesh filename=package://my_robot_description/models/upper_body.stl scale=0.4 0.4 0.4
- link base_wheel_left: geometry collision cylinder length=0.05 radius=0.104; visual mesh filename=package://my_robot_description/models/wheel_left.stl scale=0.4 0.4 0.4
- link base_wheel_right: geometry collision cylinder length=0.05 radius=0.104; visual mesh filename=package://my_robot_description/models/wheel_right.stl scale=0.4 0.4 0.4
- link camera_back: geometry visual mesh filename=package://my_robot_description/models/camera_rear.stl scale=0.4 0.4 0.4
- link camera_back_floor: geometry visual mesh filename=package://my_robot_description/models/camera_rear_bottom.stl scale=0.4 0.4 0.4
- link camera_front: geometry visual mesh filename=package://my_robot_description/models/camera_front.stl scale=0.4 0.4 0.4
- link camera_front_floor: geometry visual mesh filename=package://my_robot_description/models/camera_front_bottom.s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 scale=0.4 0.4 0.4
- link camera_left: geometry visual mesh filename=package://my_robot_description/models/camera_left.stl scale=0.4 0.4 0.4
- link camera_right: geometry visual mesh filename=package://my_robot_description/models/camera_right.stl scale=0.4 0.4 0.4
- link lidar: geometry collision cylinder length=0.016 radius=0.02; visual mesh filename=package://my_robot_description/models/lidar.stl scale=0.4 0.4 0.4
- link small_base: geometry collision box size=0.8 0.6 0.12; visual mesh filename=package://my_robot_description/models/lower_body.stl scale=0.4 0.4 0.4
- link small_base_brush_left: geometry collision cylinder length=0.02 radius=0.06; visual mesh filename=package://my_robot_description/models/brush_left.stl scale=0.4 0.4 0.4
- link small_base_brush_right: geometry collision cylinder length=0.02 radius=0.06; visual mesh filename=package://my_robot_description/models/brush_right.stl scale=0.4 0.4 0.4
- link small_base_wheel_front: geometry collision cylinder length=0.05 radius=0.104; visual mesh filename=package://my_robot_description/models/wheel_front.stl scale=0.4 0.4 0.4
Joints:
- joint brush_left_to_small_base: axis 0 0 1 -> 0 0 1.0
- joint brush_right_to_small_base: axis 0 0 1 -> 0 0 1.0
- joint small_base_to_base: axis 0 0 1 -> 0 0 1.0
- joint wheel_front_to_small_base: axis 0 1 0 -> 0 1.0 0
- joint wheel_left_to_base: axis 0 1 0 -> 0 1.0 0
- joint wheel_right_to_base: axis 0 1 0 -> 0 1.0 0
